File: chandelierLEDPCB/chandelierLEDPCB.kicad_pcb (KiCad board)
At the start: 2 copper layers, 102 x 102 mm, 122 parts, among them J1 JST PH 1x02 SMT VERT, J3 JST PH 1x02 SMT VERT, Q1 Si2301CDS, Q10 Si2301CDS, Q11 Si2301CDS, Q12 Si2301CDS, Q13 Si2301CDS, Q14 Si2301CDS, Q15 Si2301CDS, Q16 Si2301CDS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

Commit message: Changed board outline
Other:
- board size 102 x 102 mm -> 100 x 100 mm
